File: kicad/keyboard/keyboard.kicad_pcb (KiCad board)
At the start: 2 copper layers, 143.5 x 97 mm, 32 parts

Commit message: ajout des trous de vis
Parts:
- added _1: , MountingHole_2.2mm_M2_Pad_Via, F.Cu at (145.5, 104.0)
- added _2: , MountingHole_2.2mm_M2_Pad_Via, F.Cu at (236.0, 102.5)
- added _3: , MountingHole_2.2mm_M2_Pad_Via, F.Cu at (235.5, 161.0)
- added _4: , MountingHole_2.2mm_M2_Pad_Via, F.Cu at (155.0, 150.0)
- added _5: , MountingHole_2.2mm_M2_Pad_Via, F.Cu at (191.8, 122.0)
- moved REF** 0.50 mm to (253.7, 131.0)

Commit message: ajustement de la footprint
Parts:
- removed the REF** at (194.8, 112.0)
- removed the REF** at (226.5, 93.0)
- removed the REF** at (232.8, 112.0)
- removed the REF** at (131.5, 93.0)
- removed the REF** at (207.5, 93.0)
- removed the REF** at (182.2, 131.0)
- removed the REF** at (175.8, 112.0)
- removed the REF** at (245.5, 93.0)
- removed the REF** at (169.5, 93.0)
- removed the REF** at (201.2, 131.0)
- removed the REF** at (239.2, 131.0)
- removed the REF** at (156.8, 112.0)
- removed the REF** at (220.2, 131.0)
- removed the REF** at (137.8, 131.0)
- removed the REF** at (213.8, 112.0)
- removed the REF** at (150.5, 93.0)
- removed the REF** at (134.7, 112.0)
- removed the REF** at (163.2, 131.0)
- removed the REF** at (188.5, 93.0)
- added REF**: HESwitch_Michka, HESwitch_Michka, B.Cu at (182.2, 131.0)
- added REF**: HESwitch_Michka, HESwitch_Michka, B.Cu at (175.8, 112.0)
- added REF**: HESwitch_Michka, HESwitch_Michka, B.Cu at (169.5, 93.0)
- added REF**: HESwitch_Michka, HESwitch_Michka, B.Cu at (201.2, 131.0)
- added REF**: HESwitch_Michka, HESwitch_Michka, B.Cu at (194.8, 112.0)
- added REF**: HESwitch_Michka, HESwitch_Michka, B.Cu at (188.5, 93.0)
- added REF**: HESwitch_Michka, HESwitch_Michka, B.Cu at (220.2, 131.0)
- added REF**: HESwitch_Michka, HESwitch_Michka, B.Cu at (213.8, 112.0)
- added REF**: HESwitch_Michka, HESwitch_Michka, B.Cu at (137.8, 131.0)
- added REF**: HESwitch_Michka, HESwitch_Michka, B.Cu at (207.5, 93.0)
- added REF**: HESwitch_Michka, HESwitch_Michka, B.Cu at (239.2, 131.0)
- added REF**: HESwitch_Michka, HESwitch_Michka, B.Cu at (232.8, 112.0)
- added REF**: HESwitch_Michka, HESwitch_Michka, B.Cu at (226.5, 93.0)
- added REF**: HESwitch_Michka, HESwitch_Michka, B.Cu at (245.5, 93.0)
- added REF**: HESwitch_Michka, HESwitch_Michka, B.Cu at (134.7, 112.0)
- added REF**: HESwitch_Michka, HESwitch_Michka, B.Cu at (131.5, 93.0)
- added REF**: HESwitch_Michka, HESwitch_Michka, B.Cu at (163.2, 131.0)
- added REF**: HESwitch_Michka, HESwitch_Michka, B.Cu at (156.8, 112.0)
- added REF**: HESwitch_Michka, HESwitch_Michka, B.Cu at (150.5, 93.0)
- moved _2 0.50 mm to (236.0, 102.0)
- turned REF** to 180 degrees
Connections:
- REF** pad 1: (no net) -> GND (x11)
- REF** pad 2: col0_r4 -> VCC
- REF** pad 2: col3_r4 -> VCC
- REF** pad 2: col4_r4 -> VCC
- REF** pad 2: col5_r4 -> VCC
- REF** pad 2: col0_r5 -> VCC
- REF** pad 2: col1_r5 -> VCC
- REF** pad 2: col2_r5 -> VCC
- REF** pad 2: col3_r5 -> VCC
- REF** pad 2: col4_r5 -> VCC
- REF** pad 2: col1_r4 -> VCC
- REF** pad 2: col2_r4 -> VCC
Other:
- net class Default added: clearance 0.2, trace_width 0.25, via_dia 0.8, via_drill 0.4
