File: ergogen/output/pcbs/first.kicad_pcb (KiCad board)
At the start: 2 copper layers, 143.5 x 97 mm, 37 parts

Commit message: ajustement du layout mcu et mux ergogen
Connections:
- REF** pad 1: col4_r2 -> thumb2_r5
- REF** pad 2: col3_r2 -> thumb3_r5
- REF** pad 25: col3_r3 -> col0_r2
- REF** pad 26: col4_r3 -> col1_r2
- REF** pad 27: col5_r3 -> col2_r2
- REF** pad 28: col0_r4 -> col3_r2
- REF** pad 29: col1_r4 -> col4_r2
- REF** pad 3: col2_r2 -> thumb4_r5
- REF** pad 30: col2_r4 -> col5_r2
- REF** pad 31: col3_r4 -> col0_r3
- REF** pad 32: col4_r4 -> col1_r3
- REF** pad 33: col5_r4 -> col2_r3
- REF** pad 34: thumb0_r5 -> col3_r3
- REF** pad 35: thumb1_r5 -> col4_r3
- REF** pad 36: thumb2_r5 -> col5_r3
- REF** pad 37: thumb3_r5 -> col0_r4
- REF** pad 38: thumb4_r5 -> col1_r4
- REF** pad 39: (no net) -> col2_r4
- REF** pad 4: col1_r2 -> (no net)
- REF** pad 40: (no net) -> col3_r4
- REF** pad 45: col2_r3 -> col4_r4
- REF** pad 46: col1_r3 -> col5_r4
- REF** pad 47: col0_r3 -> thumb0_r5
- REF** pad 48: col5_r2 -> thumb1_r5
- REF** pad 5: col0_r2 -> (no net)
- REF** pad 27: (no net) -> AIN1
- REF** pad 30: (no net) -> VCC
- REF** pad 31: (no net) -> GND
- REF** pad 5: MUX_CS -> (no net)
- REF** pad 6: MUX_WR -> (no net)
- REF** pad 7: MUX_EN -> (no net)
- REF** pad 8: MUX_D -> (no net)

Commit message: miroir y ADG732/arangement.py/mv footprint footprints
Parts:
- added REF**: C_0805_2012Metric, C_0805_2012Metric, F.Cu at (0.00, 0.00)
Other:
- board size 143.5 x 97 mm -> 143.7 x 97.2 mm
