File: ergogen/output/pcbs/first.kicad_pcb (KiCad board)
At the start: 2 copper layers, 143.7 x 97.2 mm, 38 parts

Commit message: connexion mux
Parts:
- turned REF** to 0 degrees
Connections:
- REF** pad 1: thumb2_r5 -> col5_r3
- REF** pad 10: col2_r1 -> col3_r2
- REF** pad 11: col1_r1 -> col4_r2
- REF** pad 12: col0_r1 -> col5_r2
- REF** pad 2: thumb3_r5 -> col4_r3
- REF** pad 25: col0_r2 -> col0_r1
- REF** pad 26: col1_r2 -> col1_r1
- REF** pad 27: col2_r2 -> col2_r1
- REF** pad 28: col3_r2 -> col3_r1
- REF** pad 29: col4_r2 -> col4_r1
- REF** pad 3: thumb4_r5 -> col3_r3
- REF** pad 30: col5_r2 -> col5_r1
- REF** pad 31: col0_r3 -> col6_r1
- REF** pad 32: col1_r3 -> (no net)
- REF** pad 33: col2_r3 -> (no net)
- REF** pad 34: col3_r3 -> col4_r5
- REF** pad 35: col4_r3 -> col3_r5
- REF** pad 36: col5_r3 -> col2_r5
- REF** pad 37: col0_r4 -> col1_r5
- REF** pad 38: col1_r4 -> col0_r5
- REF** pad 39: col2_r4 -> col5_r4
- REF** pad 4: (no net) -> col2_r3
- REF** pad 40: col3_r4 -> col4_r4
- REF** pad 45: col4_r4 -> col3_r4
- REF** pad 46: col5_r4 -> col2_r4
- REF** pad 47: thumb0_r5 -> col1_r4
- REF** pad 48: thumb1_r5 -> col0_r4
- REF** pad 5: (no net) -> col1_r3
- REF** pad 6: col6_r1 -> col0_r3
- REF** pad 7: col5_r1 -> col0_r2
- REF** pad 8: col4_r1 -> col1_r2
- REF** pad 9: col3_r1 -> col2_r2
- REF** pad 0: MUX_A0 -> MUX_A4
- REF** pad 1: MUX_A1 -> MUX_A3
- REF** pad 3: MUX_A3 -> MUX_A1
- REF** pad 4: MUX_A4 -> MUX_A0
