File: ergogen/output/pcbs/first.kicad_pcb (KiCad board)
At the start: 2 copper layers, 143.7 x 97.2 mm, 38 parts

Commit message: passage kicad
Parts:
- removed the REF** at (0.00, 0.00)
Other:
- board size 143.7 x 97.2 mm -> 143.5 x 97 mm
Changed lines of the file:
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@@
       (pad "1" thru_hole circle locked (at 0 -1.65) (size 0.7 0.7) (drill 0.4) (layers *.Cu *.Mask))
     )
-		(footprint "C_0805_2012Metric"
-			(version 20260206)
-			(generator "kicad-footprint-generator")
-			(layer "F.Cu")
-			(descr "Capacitor SMD 0805 (2012 Metric), square (rectangular) end terminal, IPC-7351 nominal, (Body size source: IPC-SM-782 page 76, https://www.pcb-3d.com/wordpress/wp-content/uploads/ipc-sm-782a_amendment_1_and_2.pdf, https://docs.google.com/spreadsheets/d/1BsfQQcO9C6DZCsRaXUlFlo91Tg2WpOkGARC1WS5S8t0/edit?usp=sharing)")
-			(tags "capacitor")
-			(property "Reference" "REF**"
-				(at 0 -1.68 0)
-				(layer "F.SilkS")
-				(effects
-					(font
-						(size 1 1)
-						(thickness 0.15)
-					)
-				)
-			)
-			(property "Value" "C_0805_2012Metric"
-				(at 0 1.68 0)
-				(layer "F.Fab")
-				(effects
-					(font
-						(size 1 1)
-						(thickness 0.15)
-					)
-				)
-			)
-			(property "KiLib_Generator" "SMD_2terminal_chip_molded"
-				(at 0 0 0)
-				(layer "F.SilkS")
-				(hide yes)
-				(effects
-					(font
-						(size 1 1)
-						(thickness 0.15)
-					)
-				)
-			)
-			(attr smd)
-			(duplicate_pad_numbers_are_jumpers no)
-			(fp_line
-				(start -0.261252 -0.735)
-				(end 0.261252 -0.735)
-				(stroke
-					(width 0.12)
-					(type solid)
-				)
-				(layer "F.SilkS")
-			)
-			(fp_line
-				(start -0.261252 0.735)
-				(end 0.261252 0.735)
-				(stroke
-					(width 0.12)
-					(type solid)
-				)
-				(layer "F.SilkS")
-			)
-			(fp_rect
-				(start -1.7 -0.98)
-				(end 1.7 0.98)
-				(stroke
-					(width 0.05)
-					(type solid)
-				)
-				(fill no)
-				(layer "F.CrtYd")
-			)
-			(fp_rect
-				(start -1 -0.625)
-				(end 1 0.625)
-				(stroke
-					(width 0.1)
-					(type solid)
-				)
-				(fill no)
-				(layer "F.Fab")
-			)
-			(fp_text user "C1"
-				(at 0 0 0)
-				(layer "F.Fab")
-				(effects
-					(font
-						(size 0.5 0.5)
-						(thickness 0.08)
-					)
-				)
-			)
-			(pad "1" smd roundrect
-				(at -0.95 0)
-				(size 1 1.45)
-				(layers "F.Cu" "F.Mask" "F.Paste")
-				(roundrect_rratio 0.25)
-				(net 2 "VCC")
-			)
-			(pad "2" smd roundrect
-				(at 0.95 0)
-				(size 1 1.45)
-				(layers "F.Cu" "F.Mask" "F.Paste")
-				(roundrect_rratio 0.25)
-				(net 1 "GND")
-			)
-			(embedded_fonts no)
-		)
     (footprint "ADG732_TQFP"
       (layer "B.Cu")
@@
 (gr_line (start 264.5000001 84.5) (end 264.5000001 177.5) (angle 90) (layer Edge.Cuts) (width 0.15))
 (gr_line (start 262.5000001 179.5) (end 123 179.5) (angle 90) (layer Edge.Cuts) (width 0.15))
-(gr_arc (start 123.0 82.5) (mid 121.5858 83.0858) (end 123.0 84.5) (layer Edge.Cuts) (width 0.15))
-(gr_arc (start 264.5000001 84.5) (mid 263.9142 83.0858) (end 262.5000001 84.5) (layer Edge.Cuts) (width 0.15))
-(gr_arc (start 262.5000001 179.5) (mid 263.9142 178.9142) (end 262.5000001 177.5) (layer Edge.Cuts) (width 0.15))
-(gr_arc (start 121.0 177.5) (mid 121.5858 178.9142) (end 123.0 177.5) (layer Edge.Cuts) (width 0.15))
+(gr_arc (start 123 84.5) (end 123 82.5) (angle -90) (layer Edge.Cuts) (width 0.15))
+(gr_arc (start 262.5000001 84.5) (end 264.5000001 84.5) (angle -90) (layer Edge.Cuts) (width 0.15))
+(gr_arc (start 262.5000001 177.5) (end 262.5000001 179.5) (angle -90) (layer Edge.Cuts) (width 0.15))
+(gr_arc (start 123 177.5) (end 121 177.5) (angle -90) (layer Edge.Cuts) (width 0.15))
 )
