File: kicad/pcb/KB-Michka-30HE.kicad_pcb (KiCad board)
At the start: 2 copper layers, 143.5 x 97 mm, 37 parts

Commit message: début routage
Parts:
- added 100nF: C_0805_2012Metric_Pad1.18x1.45mm_HandSolder, Capacitor_SMD:C_0805_2012Metric_Pad1.18x1.45mm_HandSolder, B.Cu at (259.5, 96.5)
- added 100nF: C_0805_2012Metric_Pad1.18x1.45mm_HandSolder, Capacitor_SMD:C_0805_2012Metric_Pad1.18x1.45mm_HandSolder, B.Cu at (259.0, 110.5)
- added 100µF: C_0805_2012Metric_Pad1.18x1.45mm_HandSolder, Capacitor_SMD:C_0805_2012Metric_Pad1.18x1.45mm_HandSolder, B.Cu at (259.5, 93.5)
- added 100µF: C_0805_2012Metric_Pad1.18x1.45mm_HandSolder, Capacitor_SMD:C_0805_2012Metric_Pad1.18x1.45mm_HandSolder, B.Cu at (259.0, 107.5)
- added FB: C_0805_2012Metric_Pad1.18x1.45mm_HandSolder, Capacitor_SMD:C_0805_2012Metric_Pad1.18x1.45mm_HandSolder, B.Cu at (257.5, 100.5)
Routing:
- net GND: track 0.00 -> 333.2 mm, vias 0 -> 8
- net VCC: track 0.00 -> 224.0 mm
- net MUX_A4: track 0.00 -> 12.2 mm
- net MUX_A3: track 0.00 -> 10.2 mm
- net MUX_A2: track 0.00 -> 9.14 mm
- net col0_r1: track 0.00 -> 9.11 mm, vias 0 -> 2
- net col1_r1: track 0.00 -> 8.91 mm, vias 0 -> 2
- net col2_r1: track 0.00 -> 8.70 mm, vias 0 -> 2
- net col3_r1: track 0.00 -> 8.49 mm, vias 0 -> 2
- net col6_r1: track 0.00 -> 8.49 mm, vias 0 -> 2
- net col5_r1: track 0.00 -> 8.29 mm, vias 0 -> 2
- net col4_r1: track 0.00 -> 8.29 mm, vias 0 -> 2
- net MUX_A1: track 0.00 -> 8.18 mm
- net MUX_A0: track 0.00 -> 7.33 mm
- net Q_col6_r1: track 0.00 -> 1.78 mm
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
Commit message: Routage
Parts:
- added REF**: C_0805_2012Metric_Pad1.18x1.45mm_HandSolder, Capacitor_SMD:C_0805_2012Metric_Pad1.18x1.45mm_HandSolder, B.Cu at (249.0, 125.0)
Connections:
- 100nF pad 2: VCC -> 3V3A
- 100µF pad 2: VCC -> 3V3A
- FB pad 2: VCC -> 3V3A
- REF** pad 2: VCC -> 3V3A (x30)
- REF** pad 1: col5_r3 -> col0_r3
- REF** pad 13: VCC -> 3V3A
- REF** pad 14: VCC -> 3V3A
- REF** pad 2: col4_r3 -> col1_r3
- REF** pad 25: col0_r1 -> col6_r1
- REF** pad 26: col1_r1 -> col5_r1
- REF** pad 27: col2_r1 -> col4_r1
- REF** pad 29: col4_r1 -> col2_r1
- REF** pad 3: col3_r3 -> col2_r3
- REF** pad 30: col5_r1 -> col1_r1
- REF** pad 31: col6_r1 -> col0_r1
- REF** pad 4: col2_r3 -> col3_r3
- REF** pad 5: col1_r3 -> col4_r3
- REF** pad 6: col0_r3 -> col5_r3
Routing:
- net 3V3A: track 0.00 -> 992.2 mm
- net GND: track 333.2 -> 1068.1 mm, vias 8 -> 30
- net VCC: track 224.0 -> 9.26 mm
- net col0_r5: track 0.00 -> 159.6 mm
- net col0_r1: track 9.11 -> 164.7 mm
- net col1_r5: track 0.00 -> 140.4 mm
- net col1_r1: track 8.91 -> 145.1 mm
- net col0_r2: track 0.00 -> 127.5 mm
- net col0_r4: track 0.00 -> 127.4 mm
- net col2_r5: track 0.00 -> 119.7 mm
- net col0_r3: track 0.00 -> 119.5 mm
- net col2_r1: track 8.70 -> 126.1 mm
- net col1_r2: track 0.00 -> 105.4 mm
- net col1_r4: track 0.00 -> 99.5 mm
- net col3_r1: track 8.49 -> 107.2 mm
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
Commit message: modification mineur
Routing:
- net GND: track 1068.1 -> 1036.0 mm
- net AIN1: track 45.6 -> 46.4 mm

Commit message: Routage terminé, DRC clean
Routing:
- net GND: track 1036.0 -> 1068.1 mm
- net col0_r5: track 159.6 -> 161.6 mm
- net AIN1: track 46.4 -> 45.6 mm
