File: kicad/pcb/KB-Michka-30HE.kicad_pcb (KiCad board)
At the start: 2 copper layers, 143.5 x 97 mm, 43 parts

Commit message: plan de masse
Routing:
- added copper zone on F.Cu, net GND
Changed lines of the file:
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@@
 		(net "Q_col1_r4")
+	)
+	(zone
+		(net "GND")
+		(layer "F.Cu")
+		(hatch edge 0.5)
+		(connect_pads
+			(clearance 0.508)
+		)
+		(min_thickness 0.25)
+		(fill yes
+			(thermal_gap 0.5)
+			(thermal_bridge_width 0.5)
+			(island_removal_mode 0)
+		)
+		(polygon
+			(pts
+				(xy 124 176) (xy 124 107) (xy 231 107) (xy 231 122) (xy 254 145) (xy 254 176)
+			)
+		)
 	)
 	(embedded_fonts no)
